File: pcb/whackberry_mobo/whackberry_mobo.kicad_pcb (KiCad board)
At the start: 2 copper layers, 14 parts, among them J1 GroveFemaleHeader_114020164, J2 USBa_Port_87583-0010BHLF, SW1 SW_Omron_B3FS, SW2 SW_Omron_B3FS, U2 TSOP348xx, U5 2232_display

Commit message: Ready for tracing PCB
Parts:
- moved USB-C 37.6 mm to (55.1, 72.9), turned to -90 degrees
- moved QTpy 30.3 mm to (37.2, 37.1), turned to -90 degrees
- moved R1 27.8 mm to (122.6, 54.5)
- moved IR-Re 22.0 mm to (70.5, 29.4), turned to 180 degrees
- moved RPi-Zero 10.6 mm to (65.1, 63.5)
- moved USB-A 9.55 mm to (99.0, 48.5)
- moved IR-LED 5.90 mm to (69.1, 42.0)
- moved Camera 2.00 mm to (109.4, 34.1)
- renumbered S1 to 5WayNav, U4 to Camera, U6 to CardKB, J1 to GROVE, D1 to IR-LED, U2 to IR-Re, U5 to LCD, U3 to QTpy, U1 to RPi-Zero, J2 to USB-A, U7 to USB-C
Other:
- board outline added: 121.5 x 150 mm
- board text added: "+---AirGap---"
- board text added: "+---AirGap------AirGap-----------"
- board text added: "------------AirGap------AirGap---+"
- board text added: "--------AirGap"
- board text added: "---AirGap---"
- board text added: "---AirGap---+"
- board text added: "AirGap--------"
- board text added: "Power only"

Commit message: More changes before tracing PCB
Parts:
- moved RPi-Zero 1.05 mm to (66.1, 63.3)
Other:
- outline, holes or cut-outs redrawn
- board text added: "whackberry v0.1"

Commit message: adding gerber files
Parts:
- moved R1 0.50 mm to (122.1, 54.5)
Routing:
- net Net-(GROVE-1-GND): track 0.00 -> 294.0 mm, vias 0 -> 6
- net Net-(USB-A-1-5V): track 0.00 -> 238.6 mm, vias 0 -> 5
- net Net-(GROVE-1-3.3V): track 0.00 -> 186.4 mm, vias 0 -> 6
- net Net-(5WayNav-1-CENTER): track 0.00 -> 134.1 mm, vias 0 -> 6
- net Net-(RPi-Zero-1-Pad29): track 0.00 -> 125.3 mm, vias 0 -> 4
- net Net-(5WayNav-1-COMMON): track 0.00 -> 116.2 mm
- net Net-(GROVE-1-SCL): track 0.00 -> 95.4 mm, vias 0 -> 2
- net Net-(GROVE-1-SDA): track 0.00 -> 93.6 mm
- net Net-(USB-A-1-D+): track 0.00 -> 93.5 mm, vias 0 -> 2
- net Net-(USB-A-1-D-): track 0.00 -> 90.7 mm, vias 0 -> 2
- net Net-(5WayNav-1-D): track 0.00 -> 89.8 mm, vias 0 -> 4
- net Net-(5WayNav-1-C): track 0.00 -> 80.9 mm, vias 0 -> 2
- net Net-(5WayNav-1-B): track 0.00 -> 78.4 mm, vias 0 -> 2
- net Net-(5WayNav-1-A): track 0.00 -> 76.2 mm, vias 0 -> 2
- net Net-(IR-LED-1-K): track 0.00 -> 48.6 mm, vias 0 -> 2
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Other:
- outline, holes or cut-outs redrawn

Commit message: New PCB changes(v0.2)
Other:
- outline, holes or cut-outs redrawn
- board text added: "whackberry v0.2"
- board text removed: "whackberry v0.1"
Changed lines of the file:
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@@
 		(at 109.4 34.1)
 		(property "Reference" "Camera"
-			(at 22.5 3.5 180)
+			(at 21.6 -9.1 180)
 			(unlocked yes)
 			(layer "B.SilkS")
@@
 		(pad "" np_thru_hole circle
 			(at 12.4 -11.6 90)
-			(size 2.2 2.2)
-			(drill 2.2)
+			(size 1.5 1.5)
+			(drill 2.75)
 			(layers "F&B.Cu" "*.Mask")
-			(solder_mask_margin 1.27)
+			(solder_mask_margin 1.625)
 		)
 		(pad "" np_thru_hole circle
 			(at 12.4 2.9 90)
-			(size 2.2 2.2)
-			(drill 2.2)
+			(size 1.5 1.5)
+			(drill 2.75)
 			(layers "F&B.Cu" "*.Mask")
-			(solder_mask_margin 1.27)
+			(solder_mask_margin 1.625)
 		)
 		(pad "" np_thru_hole circle
 			(at 32.6 -11.6 90)
-			(size 2.2 2.2)
-			(drill 2.2)
+			(size 1.5 1.5)
+			(drill 2.75)
 			(layers "F&B.Cu" "*.Mask")
-			(solder_mask_margin 1.27)
+			(solder_mask_margin 1.625)
 		)
 		(pad "" np_thru_hole circle
 			(at 32.6 2.9 90)
-			(size 2.2 2.2)
-			(drill 2.2)
+			(size 1.5 1.5)
+			(drill 2.75)
 			(layers "F&B.Cu" "*.Mask")
-			(solder_mask_margin 1.27)
+			(solder_mask_margin 1.625)
 		)
 	)
@@
 	)
 	(gr_circle
+		(center 42.625 165)
+		(end 45.625 165)
+		(stroke
+			(width 0)
+			(type solid)
+		)
+		(fill solid)
+		(layer "B.Mask")
+	)
+	(gr_circle
 		(center 116 23)
 		(end 119 23)
@@
 		(layer "F.Mask")
 	)
+	(gr_circle
+		(center 42.625 165)
+		(end 45.625 165)
+		(stroke
+			(width 0)
+			(type solid)
+		)
+		(fill solid)
+		(layer "F.Mask")
+	)
 	(gr_line
 		(start 148 147.4)
@@
 		(layer "Edge.Cuts")
 	)
+	(gr_circle
+		(center 42.625 165)
+		(end 44 165)
+		(stroke
+			(width 0.05)
+			(type default)
+		)
+		(fill none)
+		(layer "Edge.Cuts")
+	)
 	(gr_line
 		(start 74 21)
@@
 		(layer "Edge.Cuts")
 	)
+	(gr_circle
+		(center 131.855 34.7)
+		(end 137.855 34.7)
+		(stroke
+			(width 0.05)
+			(type default)
+		)
+		(fill none)
+		(layer "Edge.Cuts")
+	)
 	(gr_line
 		(start 86 40)
@@
 		)
 	)
-	(gr_text "whackberry v0.1"
+	(gr_text "whackberry v0.2"
 		(at 143 163 0)
 		(layer "F.SilkS")

Commit message: adding hole to access QTpy Reset button
Routing:
- net Net-(USB-A-1-5V): track 238.6 -> 243.9 mm
- net Net-(GROVE-1-GND): track 294.0 -> 298.8 mm
- net Net-(IR-Re-1-Vs): track 24.4 -> 28.6 mm
- net Net-(IR-Re-1-OUT): track 27.0 -> 30.9 mm
Other:
- outline, holes or cut-outs redrawn
- board text added: "Reset"
Changed lines of the file:
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@@
 		(at 37.18 37.12 -90)
 		(property "Reference" "QTpy"
-			(at 0 -12.7 90)
+			(at -0.12 -8.82 90)
 			(unlocked yes)
 			(layer "B.SilkS")
@@
 		(layer "Edge.Cuts")
 	)
+	(gr_circle
+		(center 56 40)
+		(end 56 43)
+		(stroke
+			(width 0.05)
+			(type default)
+		)
+		(fill none)
+		(layer "Edge.Cuts")
+	)
 	(gr_line
 		(start 38 46)
@@
 		)
 	)
+	(gr_text "Reset"
+		(at 58 36.5 0)
+		(layer "B.SilkS")
+		(effects
+			(font
+				(size 1 1)
+				(thickness 0.1)
+			)
+			(justify left bottom mirror)
+		)
+	)
 	(gr_text "--------AirGap"
 		(at 73 23.5 270)
@@
 	)
 	(segment
-		(start 48 43)
-		(end 64 27)
-		(width 0.2)
-		(layer "B.Cu")
-		(net 12)
-	)
-	(segment
 		(start 54 63.78)
 		(end 50 67.78)
@@
 	)
 	(segment
-		(start 46.54 43)
-		(end 48 43)
+		(start 66 25)
+		(end 64 27)
 		(width 0.2)
 		(layer "B.Cu")
@@
 	)
 	(segment
-		(start 66 25)
-		(end 64 27)
+		(start 64 27)
+		(end 58 33)
 		(width 0.2)
 		(layer "B.Cu")
@@
 	)
 	(segment
-		(start 63.566346 51)
-		(end 63 51)
+		(start 44.8 44.74)
+		(end 44.8 36.634315)
 		(width 0.2)
 		(layer "B.Cu")
@@
 	)
 	(segment
-		(start 94.14 47)
-		(end 84 47)
+		(start 63.566346 51)
+		(end 63 51)
 		(width 0.2)
 		(layer "B.Cu")
@@
 	)
 	(segment
-		(start 44.8 44.74)
-		(end 46.54 43)
+		(start 94.14 47)
+		(end 84 47)
 		(width 0.2)
 		(layer "B.Cu")
@@
 	)
 	(segment
+		(start 44.8 36.634315)
+		(end 48.434315 33)
+		(width 0.2)
+		(layer "B.Cu")
+		(net 12)
+	)
+	(segment
 		(start 54 67)
 		(end 54 63.78)
@@
 	)
 	(segment
+		(start 48.434315 33)
+		(end 49 33)
+		(width 0.2)
+		(layer "B.Cu")
+		(net 12)
+	)
+	(segment
 		(start 80 47)
 		(end 84 47)
@@
 	)
 	(segment
+		(start 58 33)
+		(end 49 33)
+		(width 0.2)
+		(layer "B.Cu")
+		(net 12)
+	)
+	(segment
 		(start 157.524 38.5014)
 		(end 157.524 40.476)
@@
 	)
 	(segment
+		(start 63.62 31)
+		(end 62 31)
+		(width 0.2)
+		(layer "B.Cu")
+		(net 14)
+	)
+	(segment
 		(start 49.88 44.74)
-		(end 63.62 31)
+		(end 49.88 38.12)
+		(width 0.2)
+		(layer "B.Cu")
+		(net 14)
+	)
+	(segment
+		(start 58 35)
+		(end 53 35)
 		(width 0.2)
 		(layer "B.Cu")
@@
 	)
 	(segment
+		(start 62 31)
+		(end 58 35)
+		(width 0.2)
+		(layer "B.Cu")
+		(net 14)
+	)
+	(segment
+		(start 49.88 38.12)
+		(end 53 35)
+		(width 0.2)
+		(layer "B.Cu")
+		(net 14)
+	)
+	(segment
+		(start 62.68 29.4)
+		(end 65.42 29.4)
+		(width 0.2)
+		(layer "B.Cu")
+		(net 15)
+	)
+	(segment
+		(start 62.6 29.4)
+		(end 58 34)
+		(width 0.2)
+		(layer "B.Cu")
+		(net 15)
+	)
+	(segment
 		(start 47.34 44.74)
-		(end 62.68 29.4)
+		(end 47.34 37.66)
+		(width 0.2)
+		(layer "B.Cu")
+		(net 15)
+	)
+	(segment
+		(start 58 34)
+		(end 51 34)
+		(width 0.2)
+		(layer "B.Cu")
+		(net 15)
+	)
+	(segment
+		(start 47.34 37.66)
+		(end 51 34)
 		(width 0.2)
 		(layer "B.Cu")
@@
 	(segment
 		(start 62.68 29.4)
-		(end 65.42 29.4)
+		(end 62.6 29.4)
 		(width 0.2)
 		(layer "B.Cu")
@@
 	)
 	(segment
-		(start 48 42)
-		(end 66 24)
-		(width 0.2)
-		(layer "B.Cu")
-		(net 16)
-	)
-	(segment
 		(start 63.24 52)
 		(end 77 52)
@@
 	)
 	(segment
-		(start 42.26 44.74)
-		(end 45 42)
+		(start 58 32)
+		(end 46 32)
 		(width 0.2)
 		(layer "B.Cu")
@@
 	)
 	(segment
-		(start 45 42)
-		(end 48 42)
-		(width 0.2)
-		(layer "B.Cu")
-		(net 16)
-	)
-	(segment
 		(start 77 24)
 		(end 82 29)
@@
 	)
 	(segment
+		(start 42.26 35.74)
+		(end 46 32)
+		(width 0.2)
+		(layer "B.Cu")
+		(net 16)
+	)
+	(segment
+		(start 42.26 44.74)
+		(end 42.26 35.74)
+		(width 0.2)
+		(layer "B.Cu")
+		(net 16)
+	)
+	(segment
 		(start 119 46)
 		(end 123 42)
@@
 		(width 0.2)
 		(layer "B.Cu")
+		(net 16)
+	)
+	(segment
+		(start 66 24)
+		(end 58 32)
+		(width 0.2)
+		(layer "B.Cu")

Commit message: Adding a control switch for bridge power and other pcb improvements
Parts:
- added S1: EG2208, Whackberry_Parts_Library:SW_EG2208, F.Cu at (61.5, 23.5)
- renumbered 5WayNav to 5WayNav-1, CardKB to CardKB-1, GROVE to GROVE-1, IR-LED to IR-LED-1, IR-Re to IR-Re-1, LCD to LCD-1, QTpy to QTpy-1, RPi-Zero to RPi-Zero-1, Camera to U4, USB-A to USB-A-1, USB-C to USB-C-1
Connections:
- IR-Re-1 pad 2: Net-(GROVE-1-GND) -> Net-(IR-Re-1-GND)
- QTpy-1 pad 5V: Net-(USB-A-1-5V) -> Net-(QTpy-1-Pad5V)
- QTpy-1 pad GND: Net-(GROVE-1-GND) -> Net-(IR-Re-1-GND)
Routing:
- net Net-(IR-Re-1-GND): track 0.00 -> 57.2 mm, vias 0 -> 2
- net Net-(GROVE-1-GND): track 298.8 -> 262.6 mm
- net Net-(QTpy-1-Pad5V): track 0.00 -> 35.0 mm
- net Net-(USB-A-1-5V): track 243.9 -> 209.2 mm, vias 5 -> 7
Other:
- board text added: "**Basic commands** - To start the GUI for the OS: `startx` **Password manager** - To add a password: `pass insert path/to/name` - To find a password: `pass find name` - To generate a password: `pass generate path/to/name` - To add metadata: `pass insert path/to/name.meta` (there are other oiptions, this is just a suggestion) - To send a password to the QT py, `pass show path/to/name | irs` - To e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"
- board text added: "Bridge Powered"
- board text added: "Bridge Unpowered"
